File: Pcb/kaika_clock.sch (KiCad schematic (older format))
At the start: 29 parts, among them J1 Conn_01x04, J6 Conn_01x04, SW1 SW_Push, U1 AMS1117-3.3, U2 STM32F103C8Tx, Y1 Crystal

Commit message: add symbls lib
Parts:
- removed P?: USB_C_Plug_USB2.0, Connector_USB:USB_C_Receptacle_Amphenol_12401610E4-2A_CircularHoles, symbol Connector:USB_C_Plug_USB2.0
- added R7: 10K, Resistor_SMD:R_0805_2012Metric_Pad1.20x1.40mm_HandSolder, symbol Device:R_Small
- added U4: TYPE-C-31-M-12, Kaka:USB-C_SMD-TYPE-C-31-M-12, symbol Kaka:TYPE-C-31-M-12
- BT1: renamed from BT?; footprint (none) -> Kaka:BAT-SMD_CR1220-2
- C1, C6: value C_Small -> 10uf
- C10, C13, C2, C3, C4, C5, C7, C8, C9: value C_Small -> 100nf
- J6: footprint Connector_PinHeader_2.54mm:PinHeader_1x04_P2.54mm_Vertical -> Connector_PinHeader_2.54mm:PinHeader_1x05_P2.54mm_Vertical
- R6: value R_Small -> 10K
- SW1: value SW_Push -> Reset; footprint (none) -> digikey:Switch_Tactile_THT_6x6mm
- Y1: footprint (none) -> Crystal:Crystal_SMD_HC49-SD_HandSoldering
- gave numbers to parts that had none: 1
Connections:
- wire segments 75 -> 103
Other:
- moved on the sheet: U1

Commit message: change usb to micro usb
Parts:
- removed BT1: Battery_Cell, Kaka:BAT-SMD_CR1220-2, symbol Device:Battery_Cell
- removed R6, R7: 10K, Resistor_SMD:R_0805_2012Metric_Pad1.20x1.40mm_HandSolder, symbol Device:R_Small
- removed U4: TYPE-C-31-M-12, Kaka:USB-C_SMD-TYPE-C-31-M-12, symbol Kaka:TYPE-C-31-M-12
- added U4: MICRO-USB_TH, Kaka-footprints:MICRO-USB-TH_MICRO-USB-A14, symbol Kaka:MICRO-USB_TH
- added U5: CR1220-2, Kaka-footprints:BAT-SMD_CR1220-2, symbol Kaka:CR1220-2
Connections:
- wire segments 103 -> 79
